File: Power Board/v0.3/Power Board/Power Board.sch (KiCad schematic (older format))
At the start: 1 part, among them J1 Battery In

Commit message: power board v0.3 - Raspberry Pi side only
Parts:
- added J2: Conn_01x06, symbol Connector_Generic:Conn_01x06
- added SW1: SW_Push, symbol Switch:SW_Push
- J1: footprint (none) -> xxxx; Digikey No. (none) -> WM17581-ND; Manufacturer (none) -> Molex; Part No. (none) -> 43650-0205
Connections:
- net GND: now also J2.2 (Pin_2), SW1.1
- net Soft Switch/5.1V_switched: now also J2.1 (Pin_1)
- new net Soft Switch/Power_Button: SW1.2
- new net Soft Switch/Power_Ctl_GPIO: J2.3 (Pin_3)
- new net Soft Switch/Power_Sense_GPIO: J2.4 (Pin_4)
- no-connect marks 0 -> 2
Changed lines of the file:
@@
 F 0 "J1" H 1642 2935 50  0000 C CNN
 F 1 "Battery In" H 1642 2844 50  0000 C CNN
-F 2 "" H 1750 2750 50  0001 C CNN
-F 3 "~" H 1750 2750 50  0001 C CNN
+F 2 "xxxx" H 1750 2750 50  0001 C CNN
+F 3 "https://www.molex.com/pdm_docs/sd/436500205_sd.pdf" H 1750 2750 50  0001 C CNN
+F 4 "WM17581-ND" H 0   0   50  0001 C CNN "Digikey No."
+F 5 "Molex" H 0   0   50  0001 C CNN "Manufacturer"
+F 6 "43650-0205" H 0   0   50  0001 C CNN "Part No."
 	1    1750 2750
 	-1   0    0    -1
 $EndComp
 $Comp
-L power:PWR_FLAG #FLG0101
+L power:PWR_FLAG #FLG01
 U 1 1 5C912A06
 P 2150 2650
-F 0 "#FLG0101" H 2150 2725 50  0001 C CNN
+F 0 "#FLG01" H 2150 2725 50  0001 C CNN
 F 1 "PWR_FLAG" H 2150 2823 50  0000 C CNN
 F 2 "" H 2150 2650 50  0001 C CNN
@@
 F0 "Pi_Power" 50
 F1 "Pi_Power.sch" 50
-F2 "Battery_Power" I L 4150 4150 50
-F3 "5.1V_unswitched" O R 5600 4100 50
+F2 "Battery_Power" I L 4150 3900 50
+F3 "5.1V_unswitched" O R 5600 3900 50
 $EndSheet
 $Sheet
-S 6500 3600 950  1050
+S 6500 3600 1500 1000
 U 5C958DBD
 F0 "Soft Switch" 50
 F1 "Soft_Switch.sch" 50
-F2 "5.1V_unswitched" I L 6500 4100 50
-F3 "5.1V_switched" O R 7450 3900 50
-F4 "Power_GPIO" B R 7450 4350 50
+F2 "5.1V_unswitched" I L 6500 3900 50
+F3 "5.1V_switched" O R 8000 3900 50
+F4 "Power_Ctl_GPIO" I R 8000 4300 50
+F5 "Power_Sense_GPIO" O R 8000 4400 50
+F6 "Power_Button" I L 6500 4350 50
 $EndSheet
-Wire Wire Line
-	5600 4100 6500 4100
 $Comp
-L power:PWR_FLAG #FLG?
+L power:PWR_FLAG #FLG02
 U 1 1 5C9A6A29
 P 2150 2950
-F 0 "#FLG?" H 2150 3025 50  0001 C CNN
+F 0 "#FLG02" H 2150 3025 50  0001 C CNN
 F 1 "PWR_FLAG" H 2150 3123 50  0000 C CNN
 F 2 "" H 2150 2950 50  0001 C CNN
@@
 	2150 2750 2150 2650
 Wire Wire Line
-	2150 2850 2350 2850
+	2150 2850 2500 2850
 Wire Wire Line
-	2350 2850 2350 2950
+	2500 2850 2500 2950
 Connection ~ 2150 2850
 $Comp
-L power:GND #PWR?
+L power:GND #PWR02
 U 1 1 5C9A724E
-P 2350 2950
-F 0 "#PWR?" H 2350 2700 50  0001 C CNN
-F 1 "GND" H 2355 2777 50  0000 C CNN
-F 2 "" H 2350 2950 50  0001 C CNN
-F 3 "" H 2350 2950 50  0001 C CNN
-	1    2350 2950
+P 2500 2950
+F 0 "#PWR02" H 2500 2700 50  0001 C CNN
+F 1 "GND" H 2505 2777 50  0000 C CNN
+F 2 "" H 2500 2950 50  0001 C CNN
+F 3 "" H 2500 2950 50  0001 C CNN
+	1    2500 2950
 	1    0    0    -1
 $EndComp
@@
 	2150 2750 3250 2750
 Wire Wire Line
-	3250 2750 3250 4150
+	3250 2750 3250 3900
 Wire Wire Line
-	3250 4150 4150 4150
+	3250 3900 4150 3900
 Connection ~ 2150 2750
+$Comp
+L Switch:SW_Push SW1
+U 1 1 5C990069
+P 2400 4350
+AR Path="/5C990069" Ref="SW1"  Part="1"
+AR Path="/5C958DBD/5C990069" Ref="SW?"  Part="1"
+F 0 "SW1" H 2400 4550 50  0000 C CNN
+F 1 "SW_Push" H 2400 4544 50  0001 C CNN
+F 2 "" H 2400 4550 50  0001 C CNN
+F 3 "~" H 2400 4550 50  0001 C CNN
+F 4 "CKN10053-ND" H -1350 0   50  0001 C CNN "Digikey No."
+F 5 "C&K" H -1350 0   50  0001 C CNN "Manufacturer"
+F 6 "PTS645VK39-2 LFS" H -1350 0   50  0001 C CNN "Part No."
+	1    2400 4350
+	1    0    0    -1
+$EndComp
+$Comp
+L power:GND #PWR01
+U 1 1 5C99610B
+P 2100 4450
+F 0 "#PWR01" H 2100 4200 50  0001 C CNN
+F 1 "GND" H 2105 4277 50  0000 C CNN
+F 2 "" H 2100 4450 50  0001 C CNN
+F 3 "" H 2100 4450 50  0001 C CNN
+	1    2100 4450
+	1    0    0    -1
+$EndComp
+Wire Wire Line
+	2200 4350 2100 4350
+Wire Wire Line
+	2100 4350 2100 4450
+Wire Wire Line
+	2600 4350 3750 4350
+Wire Wire Line
+	3750 4350 3750 5000
+Wire Wire Line
+	3750 5000 6000 5000
+Wire Wire Line
+	6000 5000 6000 4350
+Wire Wire Line
+	6000 4350 6500 4350
+Wire Wire Line
+	6500 3900 5600 3900
+$Comp
+L Connector_Generic:Conn_01x06 J2
+U 1 1 5C997D7E
+P 9800 4250
+F 0 "J2" H 9880 4242 50  0000 L CNN
+F 1 "Conn_01x06" H 9880 4151 50  0000 L CNN
+F 2 "" H 9800 4250 50  0001 C CNN
+F 3 "~" H 9800 4250 50  0001 C CNN
+F 4 "WM4904-ND" H 0   0   50  0001 C CNN "Digikey No."
+F 5 "Molex" H 0   0   50  0001 C CNN "Manufacturer"
+F 6 "70553-0005" H 0   0   50  0001 C CNN "Part No."
+	1    9800 4250
+	1    0    0    -1
+$EndComp
+Wire Wire Line
+	9600 4050 8850 4050
+Wire Wire Line
+	8850 4050 8850 3900
+Wire Wire Line
+	8850 3900 8000 3900
+Wire Wire Line
+	8000 4300 8850 4300
+Wire Wire Line
+	8850 4300 8850 4250
+Wire Wire Line
+	8850 4250 9600 4250
+Wire Wire Line
+	8000 4400 8950 4400
+Wire Wire Line
+	8950 4400 8950 4350
+Wire Wire Line
+	8950 4350 9600 4350
+Wire Wire Line
+	9600 4150 9500 4150
+Wire Wire Line
+	9500 4150 9500 4750
+$Comp
+L power:GND #PWR03
+U 1 1 5C99AE97
+P 9500 4750
+F 0 "#PWR03" H 9500 4500 50  0001 C CNN
+F 1 "GND" H 9505 4577 50  0000 C CNN
+F 2 "" H 9500 4750 50  0001 C CNN
+F 3 "" H 9500 4750 50  0001 C CNN
+	1    9500 4750
+	1    0    0    -1
+$EndComp
+NoConn ~ 9600 4450
+NoConn ~ 9600 4500
 $EndSCHEMATC
