File: Power Board/v0.4/Power Board/Power Board.sch (KiCad schematic (older format))
At the start: 31 parts, among them J1 Battery In, J2 JST B2PS-VH, J3 JST B2PS-VH, J4 JST B2PS-VH, J5 JST B2PS-VH, J6 JST B2PS-VH, J7 JST B2PS-VH, J9 Raspberry Pi, SW1 SW_Push

Commit message: Add 3D models for more components.
Parts:
- F1, F2, F3, F4, F5, F6: footprint Fuse:Fuse_1206_3216Metric -> Power_Board:Fuse_1206_3216Metric
Changed lines of the file:
@@
 F 0 "F6" V 7853 3400 50  0000 C CNN
 F 1 "Fuse" V 7944 3400 50  0000 C CNN
-F 2 "Fuse:Fuse_1206_3216Metric" V 7980 3400 50  0001 C CNN
+F 2 "Power_Board:Fuse_1206_3216Metric" V 7980 3400 50  0001 C CNN
 F 3 "~" H 8050 3400 50  0001 C CNN
 F 4 "F9967CT-ND" H -300 1950 50  0001 C CNN "Digikey No."
@@
 F 0 "F5" V 7853 3100 50  0000 C CNN
 F 1 "Fuse" V 7944 3100 50  0000 C CNN
-F 2 "Fuse:Fuse_1206_3216Metric" V 7980 3100 50  0001 C CNN
+F 2 "Power_Board:Fuse_1206_3216Metric" V 7980 3100 50  0001 C CNN
 F 3 "~" H 8050 3100 50  0001 C CNN
 F 4 "F9967CT-ND" H -300 1650 50  0001 C CNN "Digikey No."
@@
 F 0 "F4" V 7853 2800 50  0000 C CNN
 F 1 "Fuse" V 7944 2800 50  0000 C CNN
-F 2 "Fuse:Fuse_1206_3216Metric" V 7980 2800 50  0001 C CNN
+F 2 "Power_Board:Fuse_1206_3216Metric" V 7980 2800 50  0001 C CNN
 F 3 "~" H 8050 2800 50  0001 C CNN
 F 4 "F9967CT-ND" H -300 1350 50  0001 C CNN "Digikey No."
@@
 F 0 "F3" V 7853 2500 50  0000 C CNN
 F 1 "Fuse" V 7944 2500 50  0000 C CNN
-F 2 "Fuse:Fuse_1206_3216Metric" V 7980 2500 50  0001 C CNN
+F 2 "Power_Board:Fuse_1206_3216Metric" V 7980 2500 50  0001 C CNN
 F 3 "~" H 8050 2500 50  0001 C CNN
 F 4 "F9967CT-ND" H -300 1050 50  0001 C CNN "Digikey No."
@@
 F 0 "F2" V 7853 2200 50  0000 C CNN
 F 1 "Fuse" V 7944 2200 50  0000 C CNN
-F 2 "Fuse:Fuse_1206_3216Metric" V 7980 2200 50  0001 C CNN
+F 2 "Power_Board:Fuse_1206_3216Metric" V 7980 2200 50  0001 C CNN
 F 3 "~" H 8050 2200 50  0001 C CNN
 F 4 "F9967CT-ND" H -300 750 50  0001 C CNN "Digikey No."
@@
 F 0 "F1" V 7853 1900 50  0000 C CNN
 F 1 "Fuse" V 7944 1900 50  0000 C CNN
-F 2 "Fuse:Fuse_1206_3216Metric" V 7980 1900 50  0001 C CNN
+F 2 "Power_Board:Fuse_1206_3216Metric" V 7980 1900 50  0001 C CNN
 F 3 "~" H 8050 1900 50  0001 C CNN
 F 4 "F9967CT-ND" H -300 450 50  0001 C CNN "Digikey No."

Commit message: Update BOM.  Change R20 to 0603 package.
Parts:
- H1, H2, H3, H4: Digikey No. (none) -> -; Manufacturer (none) -> -; Part No. (none) -> -
- J9: Digikey No. (none) -> 455-2486-ND; Manufacturer (none) -> JST; Part No. (none) -> S10B-PUDSS-1(LF)(SN)
- R24: value 100k -> 100K; Digikey No. (none) -> -; Manufacturer (none) -> Yageo; Part No. (none) -> RC0603JR-07100K
Changed lines of the file:
@@
 F 2 "Connector_JST:JST_PUD_S10B-PUDSS-1_2x05_P2.00mm_Horizontal" H 8700 5850 50  0001 C CNN
 F 3 "~" H 8700 5850 50  0001 C CNN
+F 4 "455-2486-ND" H 0   0   50  0001 C CNN "Digikey No."
+F 5 "JST" H 0   0   50  0001 C CNN "Manufacturer"
+F 6 "S10B-PUDSS-1(LF)(SN)" H 0   0   50  0001 C CNN "Part No."
 	1    8700 5850
 	1    0    0    -1
@@
 P 4900 3250
 F 0 "R24" H 4970 3296 50  0000 L CNN
-F 1 "100k" H 4970 3205 50  0000 L CNN
+F 1 "100K" H 4970 3205 50  0000 L CNN
 F 2 "Resistor_SMD:R_0603_1608Metric" V 4830 3250 50  0001 C CNN
 F 3 "~" H 4900 3250 50  0001 C CNN
+F 4 "-" H 0   0   50  0001 C CNN "Digikey No."
+F 5 "Yageo" H 0   0   50  0001 C CNN "Manufacturer"
+F 6 "RC0603JR-07100K" H 0   0   50  0001 C CNN "Part No."
 	1    4900 3250
 	1    0    0    -1
@@
 F 2 "MountingHole:MountingHole_2.7mm_M2.5" H 6350 5350 50  0001 C CNN
 F 3 "~" H 6350 5350 50  0001 C CNN
+F 4 "-" H 0   0   50  0001 C CNN "Digikey No."
+F 5 "-" H 0   0   50  0001 C CNN "Manufacturer"
+F 6 "-" H 0   0   50  0001 C CNN "Part No."
 	1    6350 5350
 	1    0    0    -1
@@
 F 2 "MountingHole:MountingHole_2.7mm_M2.5" H 6350 5600 50  0001 C CNN
 F 3 "~" H 6350 5600 50  0001 C CNN
+F 4 "-" H 0   0   50  0001 C CNN "Digikey No."
+F 5 "-" H 0   0   50  0001 C CNN "Manufacturer"
+F 6 "-" H 0   0   50  0001 C CNN "Part No."
 	1    6350 5600
 	1    0    0    -1
@@
 F 2 "MountingHole:MountingHole_2.7mm_M2.5" H 6350 5850 50  0001 C CNN
 F 3 "~" H 6350 5850 50  0001 C CNN
+F 4 "-" H 0   0   50  0001 C CNN "Digikey No."
+F 5 "-" H 0   0   50  0001 C CNN "Manufacturer"
+F 6 "-" H 0   0   50  0001 C CNN "Part No."
 	1    6350 5850
 	1    0    0    -1
@@
 F 2 "MountingHole:MountingHole_2.7mm_M2.5" H 6350 6100 50  0001 C CNN
 F 3 "~" H 6350 6100 50  0001 C CNN
+F 4 "-" H 0   0   50  0001 C CNN "Digikey No."
+F 5 "-" H 0   0   50  0001 C CNN "Manufacturer"
+F 6 "-" H 0   0   50  0001 C CNN "Part No."
 	1    6350 6100
 	1    0    0    -1

Commit message: Add BOM massage script.  Add generated files: schematic PDF, BOM CSVs, Gerbers, drill file.
Parts:
- J1: Digikey No. WM17581-ND -> 455-1649-ND; Manufacturer Molex -> JST; Part No. 43650-0205 -> B3PS-VH(LF)(SN)
Changed lines of the file:
@@
 F 1 "Battery In" H 992 2094 50  0000 C CNN
 F 2 "Power_Board:JST_VH_B3PS-VH_1x03_P3.96mm_Horizontal" H 1100 2000 50  0001 C CNN
-F 3 "https://www.molex.com/pdm_docs/sd/436500205_sd.pdf" H 1100 2000 50  0001 C CNN
-F 4 "WM17581-ND" H -650 -750 50  0001 C CNN "Digikey No."
-F 5 "Molex" H -650 -750 50  0001 C CNN "Manufacturer"
-F 6 "43650-0205" H -650 -750 50  0001 C CNN "Part No."
+F 3 "" H 1100 2000 50  0001 C CNN
+F 4 "455-1649-ND" H -650 -750 50  0001 C CNN "Digikey No."
+F 5 "JST" H -650 -750 50  0001 C CNN "Manufacturer"
+F 6 "B3PS-VH(LF)(SN)" H -650 -750 50  0001 C CNN "Part No."
 	1    1100 2000
 	1    0    0    -1
