File: Power Board/v0.4/Power Board/Power_Meter.sch (KiCad schematic (older format))
At the start: 3 parts, among them U5 ADS1000

Commit message: Almost Rough Draft Done
Mostly routed but needs lots of TLC. Need to check rule definitions before DRC
Parts:
- added C30: 100nF, Capacitor_SMD:C_0603_1608Metric, symbol Device:C
- U5: footprint (none) -> Package_TO_SOT_SMD:SOT-23-6
Connections:
- net GND: now also C30.2
- net Pi_3.3V: now also C30.1
Changed lines of the file:
@@
 F 0 "U5" H 5700 4200 50  0000 C CNN
 F 1 "ADS1000" H 5700 3500 50  0000 C CNN
-F 2 "" H 5950 3850 50  0001 C CNN
-F 3 "" H 5950 3850 50  0001 C CNN
+F 2 "Package_TO_SOT_SMD:SOT-23-6" H 5950 3850 50  0000 C CNN
+F 3 "http://www.ti.com/lit/ds/symlink/ads1000.pdf" H 5950 3850 50  0001 C CNN
 	1    5950 3850
 	1    0    0    -1
@@
 	4950 3050 4900 3050
 Wire Wire Line
-	5950 3450 5950 3050
+	5950 3450 5950 3300
 Wire Wire Line
 	5950 3050 5900 3050
@@
 Wire Wire Line
 	6350 3750 6550 3750
+$Comp
+L Device:C C30
+U 1 1 5CB75E54
+P 7150 3850
+F 0 "C30" H 7265 3896 50  0000 L CNN
+F 1 "100nF" H 7265 3805 50  0000 L CNN
+F 2 "Capacitor_SMD:C_0603_1608Metric" H 7188 3700 50  0001 C CNN
+F 3 "~" H 7150 3850 50  0001 C CNN
+	1    7150 3850
+	1    0    0    -1
+$EndComp
+Wire Wire Line
+	5950 3300 7150 3300
+Wire Wire Line
+	7150 3300 7150 3700
+Connection ~ 5950 3300
+Wire Wire Line
+	5950 3300 5950 3050
+Wire Wire Line
+	7150 4000 7150 4450
+$Comp
+L power:GND #PWR0119
+U 1 1 5CB77FAB
+P 7150 4450
+F 0 "#PWR0119" H 7150 4200 50  0001 C CNN
+F 1 "GND" H 7155 4277 50  0000 C CNN
+F 2 "" H 7150 4450 50  0001 C CNN
+F 3 "" H 7150 4450 50  0001 C CNN
+	1    7150 4450
+	1    0    0    -1
+$EndComp
 $EndSCHEMATC

Commit message: Update BOM.  Change R20 to 0603 package.
Parts:
- C30: Digikey No. (none) -> -; Manufacturer (none) -> Murata; Part No. (none) -> GRM188R71C104KA01D
- R22: value 100K 1% -> 10K 1%; Digikey No. 311-100KHRCT-ND -> RNCP0603FTD10K0CT-ND; Manufacturer Yageo -> Stackpole; Part No. RC0603FR-07100KL -> RNCP0603FTD10K0
- R23: value 17.8K 1% -> 1.78K 1%; Digikey No. 311-17.8KHRCT-ND -> 311-17.8KHRCT-ND; Part No. RC0603FR-0717K8L -> RC0603FR-0717K8L
- U5: Digikey No. (none) -> 296-38847-1-ND; Manufacturer (none) -> TI; Part No. (none) -> ADS1000A0IDBVR
Changed lines of the file:
@@
 F 2 "Package_TO_SOT_SMD:SOT-23-6" H 5950 3850 50  0000 C CNN
 F 3 "http://www.ti.com/lit/ds/symlink/ads1000.pdf" H 5950 3850 50  0001 C CNN
+F 4 "296-38847-1-ND" H 0   0   50  0001 C CNN "Digikey No."
+F 5 "TI" H 0   0   50  0001 C CNN "Manufacturer"
+F 6 "ADS1000A0IDBVR" H 0   0   50  0001 C CNN "Part No."
 	1    5950 3850
 	1    0    0    -1
@@
 P 4950 3400
 F 0 "R22" H 5020 3446 50  0000 L CNN
-F 1 "100K 1%" H 5020 3355 50  0000 L CNN
+F 1 "10K 1%" H 5020 3355 50  0000 L CNN
 F 2 "Resistor_SMD:R_0603_1608Metric" V 4880 3400 50  0001 C CNN
 F 3 "~" H 4950 3400 50  0001 C CNN
-F 4 "311-100KHRCT-ND" H 0   0   50  0001 C CNN "Digikey No."
-F 5 "Yageo" H 0   0   50  0001 C CNN "Manufacturer"
-F 6 " RC0603FR-07100KL" H 0   0   50  0001 C CNN "Part No."
+F 4 "RNCP0603FTD10K0CT-ND" H 0   0   50  0001 C CNN "Digikey No."
+F 5 "Stackpole" H 0   0   50  0001 C CNN "Manufacturer"
+F 6 "RNCP0603FTD10K0" H 0   0   50  0001 C CNN "Part No."
 	1    4950 3400
 	1    0    0    -1
@@
 P 4950 4100
 F 0 "R23" H 5020 4146 50  0000 L CNN
-F 1 "17.8K 1%" H 5020 4055 50  0000 L CNN
+F 1 "1.78K 1%" H 5020 4055 50  0000 L CNN
 F 2 "Resistor_SMD:R_0603_1608Metric" V 4880 4100 50  0001 C CNN
 F 3 "~" H 4950 4100 50  0001 C CNN
-F 4 " 311-17.8KHRCT-ND" H 0   0   50  0001 C CNN "Digikey No."
+F 4 "311-17.8KHRCT-ND" H 0   0   50  0001 C CNN "Digikey No."
 F 5 "Yageo" H 0   0   50  0001 C CNN "Manufacturer"
-F 6 " RC0603FR-0717K8L " H 0   0   50  0001 C CNN "Part No."
+F 6 "RC0603FR-0717K8L" H 0   0   50  0001 C CNN "Part No."
 	1    4950 4100
 	1    0    0    -1
@@
 F 2 "Capacitor_SMD:C_0603_1608Metric" H 7188 3700 50  0001 C CNN
 F 3 "~" H 7150 3850 50  0001 C CNN
+F 4 "-" H 0   0   50  0001 C CNN "Digikey No."
+F 5 "Murata" H 0   0   50  0001 C CNN "Manufacturer"
+F 6 "GRM188R71C104KA01D" H 0   0   50  0001 C CNN "Part No."
 	1    7150 3850
 	1    0    0    -1
