File: Power Board/v0.4/Power Board/Pi_Power.sch (KiCad schematic (older format))
At the start: 23 parts, among them Q1 SI5504BDC, U1 LMZ14203

Commit message: Add ADC to monitor battery voltage.
Changed lines of the file:
@@
 $Descr USLetter 11000 8500
 encoding utf-8
-Sheet 2 4
+Sheet 2 5
 Title ""
 Date ""
@@
 Connection ~ 4800 2150
 Wire Wire Line
-	4800 2150 4300 2150
+	4800 2150 4450 2150
 Connection ~ 5150 2150
 Connection ~ 5500 2150
@@
 Text Label 4600 2150 0    50   ~ 0
 Vin_switched
+Wire Wire Line
+	4450 2150 4450 1050
+Wire Wire Line
+	4450 1050 4850 1050
+Connection ~ 4450 2150
+Wire Wire Line
+	4450 2150 4300 2150
+Text GLabel 4850 1050 2    50   Input ~ 0
+Vin_switched
 $EndSCHEMATC

Commit message: Update BOM.  Change R20 to 0603 package.
Parts:
- C10: Part No. LMK325BJ107MM-T -> LMK325BJ107MM-T
- C4, C5: Part No. GRM21BR61E106MA73L -> GRM21BR61E106MA73L
- C8: Part No. 885012206091 -> 885012206091
Changed lines of the file:
@@
 F 4 "490-10748-1-ND" H 0   0   50  0001 C CNN "Digikey No."
 F 5 "Murata" H 0   0   50  0001 C CNN "Manufacturer"
-F 6 " GRM21BR61E106MA73L " H 0   0   50  0001 C CNN "Part No."
+F 6 "GRM21BR61E106MA73L" H 0   0   50  0001 C CNN "Part No."
 	1    5250 5000
 	0    -1   -1   0
@@
 F 4 "490-10748-1-ND" H 0   0   50  0001 C CNN "Digikey No."
 F 5 "Murata" H 0   0   50  0001 C CNN "Manufacturer"
-F 6 " GRM21BR61E106MA73L " H 0   0   50  0001 C CNN "Part No."
+F 6 "GRM21BR61E106MA73L" H 0   0   50  0001 C CNN "Part No."
 	1    5150 2450
 	1    0    0    -1
@@
 F 4 "732-8009-1-ND" H 0   0   50  0001 C CNN "Digikey No."
 F 5 "Wurth" H 0   0   50  0001 C CNN "Manufacturer"
-F 6 " 885012206091" H 0   0   50  0001 C CNN "Part No."
+F 6 "885012206091" H 0   0   50  0001 C CNN "Part No."
 	1    8750 2450
 	1    0    0    -1
@@
 F 4 "587-1965-1-ND" H 550 -1250 50  0001 C CNN "Digikey No."
 F 5 "Taiyo Yuden" H 550 -1250 50  0001 C CNN "Manufacturer"
-F 6 " LMK325BJ107MM-T " H 550 -1250 50  0001 C CNN "Part No."
+F 6 "LMK325BJ107MM-T" H 550 -1250 50  0001 C CNN "Part No."
 	1    9350 2450
 	1    0    0    -1

Commit message: Add BOM massage script.  Add generated files: schematic PDF, BOM CSVs, Gerbers, drill file.
Parts:
- U1: Digikey No. - -> LMZ14203TZX-ADJ/NOPBCT-ND; Part No. LMZ14203TZE-ADJ/NOPB -> LMZ14203TZX-ADJ/NOPB
Changed lines of the file:
@@
 F 4 "TI" H 850 250 50  0001 C CNN "Manufacturer"
 F 5 "TO-PMOD 7" H 850 250 50  0001 C CNN "Package"
-F 6 "LMZ14203TZE-ADJ/NOPB" H 850 250 50  0001 C CNN "Part No."
-F 7 "-" H 0   0   50  0001 C CNN "Digikey No."
+F 6 " LMZ14203TZX-ADJ/NOPB " H 850 250 50  0001 C CNN "Part No."
+F 7 "LMZ14203TZX-ADJ/NOPBCT-ND" H 0   0   50  0001 C CNN "Digikey No."
 	1    7150 2350
 	1    0    0    -1
