File: Power Board/v0.5/Power Board/Power Board.kicad_pcb (KiCad board)
At the start: 4 copper layers, 70 x 80 mm, 91 parts, among them J1 Battery In, J2 JST B2PS-VH, J3 JST B2PS-VH, J4 JST B2PS-VH, J5 JST B2PS-VH, J6 JST B2PS-VH, J7 JST B2PS-VH, J9 Raspberry Pi, Q1 SI5504BDC, SW1 SW_Push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

Commit message: Update version number on silkscreen.
Other:
- board text added: "LED Cube Power Board v0.5"
- board text removed: "LED Cube Power Board v0.4"
Changed lines of the file:
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@@
     )
   )
-  (gr_text "LED Cube Power Board v0.4" (at 85 108.75) (layer F.SilkS)
+  (gr_text "LED Cube Power Board v0.5" (at 85 108.75) (layer F.SilkS)
     (effects (font (size 1.5 1.5) (thickness 0.3)) (justify left))
   )
