File: Power Board/v0.5/Power Board/Panel_Power.sch (KiCad schematic (older format))
At the start: 27 parts, among them U2 TPS53819A, U3 CSD86360Q5D

Commit message: Correct C14 footprint, remove C6 and C9 incorrect package.
Parts:
- C14: footprint Capacitor_SMD:C_0603_1608Metric -> Capacitor_SMD:C_0805_2012Metric
Changed lines of the file:
@@
 F 0 "C14" H 3300 2350 50  0000 L CNN
 F 1 "1µF" H 3300 2150 50  0000 L CNN
-F 2 "Capacitor_SMD:C_0603_1608Metric" H 3288 2100 50  0001 C CNN
+F 2 "Capacitor_SMD:C_0805_2012Metric" H 3288 2100 50  0001 C CNN
 F 3 "~" H 3250 2250 50  0001 C CNN
 F 4 "587-1438-1-ND" H -100 0   50  0001 C CNN "Digikey No."
